Commit message: will be updated

File: ROS_learning/hrwros_ws/src/hrwros_week2_v09/hrwros_week2/urdf/hrwros_assignment1.xacro (robot description, xacro)
@@ -72,3 +72,9 @@
   </joint>
   <!-- Add your solution to assignment 1 here -->
+  <!-- bin 2 -->
+  <joint name="bin_2_joint" type="fixed">
+    <parent link="world_interface" />
+    <child link="bin_2_base_link" />
+    <origin xyz="2 2 0" rpy="0 0 0" />
+  </joint>
 </robot>

File: ROS_learning/hrwros_ws/src/hrwros_week2_v09/hrwros_week2/urdf/hrwros_assignment2.xacro (robot description, xacro)
@@ -72,3 +72,19 @@
   </joint>
   <!-- Add your solution to assignment 2 here -->
+  <link name="green_sphere_link">
+    <visual>
+      <origin xyz="0 0 0.4" />
+      <geometry>
+        <sphere radius="0.4" />
+      </geometry>
+      <material name="green_sphere_color">
+        <color rgba="0 1 0 1" />
+      </material>
+    </visual>
+  </link>
+  <joint name="green_sphere_joint" type="fixed">
+    <parent link="world_interface" />
+    <child link="green_sphere_link" />
+    <origin xyz="5 -6 0" />
+  </joint>
 </robot>

File: ROS_learning/hrwros_ws/src/hrwros_week2_v09/hrwros_week2/urdf/hrwros_assignment3.xacro (robot description, xacro)
@@ -65,7 +65,7 @@
   </joint>
   <!-- Update the below block for assignment 3 here -->
-  <xacro:include filename="$(find ur_description)/urdf/ur5.urdf.xacro"/>
-  <xacro:ur5_robot prefix="robot2_" joint_limited="true"/>
-  <joint name="robot2-robot2_pedestal_joint" type="fixed">
+  <xacro:include filename="$(find hrwros_week2)/urdf/robot/lrmate200ic_macro.xacro"/>
+  <xacro:fanuc_lrmate200ic prefix="robot2_" joint_limited="true"/>
+  <joint name="robot2-robot2_fanuc_lrmate200ic" type="fixed">
     <parent link="robot2_pedestal_link" />
     <child link="robot2_base_link" />
